File: Kicad/Neotron-Baseboard-100.kicad_pcb (KiCad board)
At the start: 2 copper layers, 0 parts

Commit message: Bring over basic PCB shape.
Dropped down to "short micro-ATX" - 9.6" across, 6.7" high.
Parts:
- added BT901: Coin Cell, Neotron-Common-Hardware:BatteryHolder_Keystone_103_1x20mm, F.Cu at (153.1, 192.5)
- added C1001: 10u, Capacitor_THT:CP_Radial_D6.3mm_P2.50mm, F.Cu at (256.0, 148.0)
- added C1002: 100n, Capacitor_SMD:C_0805_2012Metric_Pad1.15x1.40mm_HandSolder, F.Cu at (189.3, 187.7)
- added C201: 220n, Capacitor_SMD:C_0805_2012Metric_Pad1.15x1.40mm_HandSolder, F.Cu at (250.4, 85.5)
- added C202: 100n, Capacitor_SMD:C_0805_2012Metric_Pad1.15x1.40mm_HandSolder, F.Cu at (236.2, 84.5)
- added C203: 100n, Capacitor_SMD:C_0805_2012Metric_Pad1.15x1.40mm_HandSolder, F.Cu at (253.7, 79.6)
- added C204: 100n, Capacitor_SMD:C_0805_2012Metric_Pad1.15x1.40mm_HandSolder, F.Cu at (250.4, 82.6)
- added C205: 100n, Capacitor_SMD:C_0805_2012Metric_Pad1.15x1.40mm_HandSolder, F.Cu at (245.7, 85.5)
- added C206: 10u, Capacitor_THT:CP_Radial_D6.3mm_P2.50mm, F.Cu at (236.6, 79.1)
- added C301: 100n, Capacitor_SMD:C_0805_2012Metric_Pad1.15x1.40mm_HandSolder, F.Cu at (175.8, 75.0)
- added C302: 100n, Capacitor_SMD:C_0805_2012Metric_Pad1.15x1.40mm_HandSolder, F.Cu at (163.2, 71.4)
- added C303: 100n, Capacitor_SMD:C_0805_2012Metric_Pad1.15x1.40mm_HandSolder, F.Cu at (169.9, 76.5)
- added C304: 100n, Capacitor_SMD:C_0805_2012Metric_Pad1.15x1.40mm_HandSolder, F.Cu at (166.2, 71.4)
- added C305: 100n, Capacitor_SMD:C_0805_2012Metric_Pad1.15x1.40mm_HandSolder, F.Cu at (163.2, 66.6)
- added C306: 1n, Capacitor_SMD:C_0805_2012Metric_Pad1.15x1.40mm_HandSolder, F.Cu at (172.8, 76.5)
- added C307: 1n, Capacitor_SMD:C_0805_2012Metric_Pad1.15x1.40mm_HandSolder, F.Cu at (177.7, 79.8)
- added C308: 10u Low ESR, Capacitor_THT:CP_Radial_D6.3mm_P2.50mm, F.Cu at (172.3, 84.1)
- added C309: 12p, Capacitor_SMD:C_0805_2012Metric_Pad1.15x1.40mm_HandSolder, F.Cu at (169.1, 71.4)
- added C310: 10n, Capacitor_SMD:C_0805_2012Metric_Pad1.15x1.40mm_HandSolder, F.Cu at (166.2, 66.6)
- added C311: 10n, Capacitor_SMD:C_0805_2012Metric_Pad1.15x1.40mm_HandSolder, F.Cu at (163.2, 61.9)
- added C312: 12p, Capacitor_SMD:C_0805_2012Metric_Pad1.15x1.40mm_HandSolder, F.Cu at (172.1, 71.8)
- added C401: 22p, Capacitor_SMD:C_0805_2012Metric_Pad1.15x1.40mm_HandSolder, F.Cu at (177.8, 113.0)
- added C402: 10u, Capacitor_THT:CP_Radial_D6.3mm_P2.50mm, F.Cu at (178.4, 95.9)
- added C403: 10u, Capacitor_THT:CP_Radial_D6.3mm_P2.50mm, F.Cu at (151.7, 115.7)
- added C404: 10u, Capacitor_THT:CP_Radial_D6.3mm_P2.50mm, F.Cu at (165.0, 103.8)
- added C405: 22p, Capacitor_SMD:C_0805_2012Metric_Pad1.15x1.40mm_HandSolder, F.Cu at (164.1, 117.3)
- added C406: 100n, Capacitor_SMD:C_0805_2012Metric_Pad1.15x1.40mm_HandSolder, F.Cu at (179.8, 101.6)
- added C407: 10u, Capacitor_THT:CP_Radial_D6.3mm_P2.50mm, F.Cu at (138.4, 122.8)
- added C408: 100n, Capacitor_SMD:C_0805_2012Metric_Pad1.15x1.40mm_HandSolder, F.Cu at (149.8, 129.2)
- added C409: 10u, Capacitor_THT:CP_Radial_D6.3mm_P2.50mm, F.Cu at (130.4, 122.8)
- added C410: 10u, Capacitor_THT:CP_Radial_D6.3mm_P2.50mm, F.Cu at (143.8, 111.9)
- added C411: 100n, Capacitor_SMD:C_0805_2012Metric_Pad1.15x1.40mm_HandSolder, F.Cu at (166.5, 113.0)
- added C412: 10u, Capacitor_THT:CP_Radial_D6.3mm_P2.50mm, F.Cu at (157.1, 100.0)
- added C413: 100n, Capacitor_SMD:C_0805_2012Metric_Pad1.15x1.40mm_HandSolder, F.Cu at (166.5, 109.5)
- added C414: 10u, Capacitor_THT:CP_Radial_D6.3mm_P2.50mm, F.Cu at (170.4, 95.9)
- added C415: 10u, Capacitor_THT:CP_Radial_D6.3mm_P2.50mm, F.Cu at (159.7, 111.6)
- added C416: 100n, Capacitor_SMD:C_0805_2012Metric_Pad1.15x1.40mm_HandSolder, F.Cu at (127.2, 128.5)
- added C417: 10u, Capacitor_THT:CP_Radial_D6.3mm_P2.50mm, F.Cu at (143.8, 104.0)
- added C418: 470n, Capacitor_SMD:C_0805_2012Metric_Pad1.15x1.40mm_HandSolder, F.Cu at (158.5, 117.3)
- added C419: 470n, Capacitor_SMD:C_0805_2012Metric_Pad1.15x1.40mm_HandSolder, F.Cu at (144.2, 129.2)
- added C420: 220u, Capacitor_THT:CP_Radial_D6.3mm_P2.50mm, F.Cu at (154.4, 123.5)
- added C421: 220u, Capacitor_THT:CP_Radial_D6.3mm_P2.50mm, F.Cu at (173.0, 103.8)
- added C422: 470n, Capacitor_SMD:C_0805_2012Metric_Pad1.15x1.40mm_HandSolder, F.Cu at (138.5, 128.5)
- added C423: 470n, Capacitor_SMD:C_0805_2012Metric_Pad1.15x1.40mm_HandSolder, F.Cu at (132.8, 128.5)
- added C424: DNF, Capacitor_SMD:C_0805_2012Metric_Pad1.15x1.40mm_HandSolder, F.Cu at (121.5, 129.7)
- added C425: 1u, Capacitor_THT:CP_Radial_D6.3mm_P2.50mm, F.Cu at (146.4, 123.5)
- added C426: DNF, Capacitor_SMD:C_0805_2012Metric_Pad1.15x1.40mm_HandSolder, F.Cu at (121.5, 126.2)
- added C427: DNF, Capacitor_SMD:C_0805_2012Metric_Pad1.15x1.40mm_HandSolder, F.Cu at (115.9, 129.7)
- added C428: DNF, Capacitor_SMD:C_0805_2012Metric_Pad1.15x1.40mm_HandSolder, F.Cu at (115.9, 126.2)
- added C429: 47p, Capacitor_SMD:C_0805_2012Metric_Pad1.15x1.40mm_HandSolder, F.Cu at (151.7, 107.8)
- added C430: DNF, Capacitor_SMD:C_0805_2012Metric_Pad1.15x1.40mm_HandSolder, F.Cu at (172.1, 109.5)
- added C431: DNF, Capacitor_SMD:C_0805_2012Metric_Pad1.15x1.40mm_HandSolder, F.Cu at (166.8, 120.9)
- added C432: DNF, Capacitor_SMD:C_0805_2012Metric_Pad1.15x1.40mm_HandSolder, F.Cu at (177.8, 109.5)
- added C433: DNF, Capacitor_SMD:C_0805_2012Metric_Pad1.15x1.40mm_HandSolder, F.Cu at (169.8, 116.6)
- added C434: DNF, Capacitor_SMD:C_0805_2012Metric_Pad1.15x1.40mm_HandSolder, F.Cu at (161.1, 124.4)
- added C435: DNF, Capacitor_SMD:C_0805_2012Metric_Pad1.15x1.40mm_HandSolder, F.Cu at (155.4, 129.2)
- added C436: DNF, Capacitor_SMD:C_0805_2012Metric_Pad1.15x1.40mm_HandSolder, F.Cu at (179.8, 105.2)
- added C437: DNF, Capacitor_SMD:C_0805_2012Metric_Pad1.15x1.40mm_HandSolder, F.Cu at (172.1, 113.0)
- added C438: DNF, Capacitor_SMD:C_0805_2012Metric_Pad1.15x1.40mm_HandSolder, F.Cu at (161.1, 120.9)
- added C501: 100n, Capacitor_SMD:C_0805_2012Metric_Pad1.15x1.40mm_HandSolder, F.Cu at (260.3, 91.6)
- added C502: 100n, Capacitor_SMD:C_0805_2012Metric_Pad1.15x1.40mm_HandSolder, F.Cu at (220.4, 84.5)
- added C503: 4u7, Capacitor_THT:CP_Radial_D6.3mm_P2.50mm, F.Cu at (220.8, 79.1)
- added C504: 120u, Capacitor_THT:CP_Radial_D6.3mm_P2.50mm, F.Cu at (209.6, 93.1)
- added C505: 120u, Capacitor_THT:CP_Radial_D6.3mm_P2.50mm, F.Cu at (212.9, 79.1)
- added C506: 12p, Capacitor_SMD:C_0805_2012Metric_Pad1.15x1.40mm_HandSolder, F.Cu at (242.3, 54.0)
- added C507: 12p, Capacitor_SMD:C_0805_2012Metric_Pad1.15x1.40mm_HandSolder, F.Cu at (242.3, 69.3)
- added C508: 100n, Capacitor_SMD:C_0805_2012Metric_Pad1.15x1.40mm_HandSolder, F.Cu at (131.8, 71.8)
- added C509: 120u, Capacitor_THT:CP_Radial_D6.3mm_P2.50mm, F.Cu at (204.9, 79.1)
- added C510: 120u, Capacitor_THT:CP_Radial_D6.3mm_P2.50mm, F.Cu at (201.6, 93.1)
- added C511: 4u7, Capacitor_THT:CP_Radial_D6.3mm_P2.50mm, F.Cu at (136.6, 76.9)
- added C601: 100u 50V, Capacitor_THT:CP_Radial_D6.3mm_P2.50mm, F.Cu at (261.3, 109.7)
- added C602: 100u 50V, Capacitor_THT:CP_Radial_D6.3mm_P2.50mm, F.Cu at (252.7, 109.7)
- added C603: 22u, Capacitor_THT:CP_Radial_D6.3mm_P2.50mm, F.Cu at (210.3, 126.8)
- added C604: 100n, Capacitor_SMD:C_0805_2012Metric_Pad1.15x1.40mm_HandSolder, F.Cu at (228.7, 120.6)
- added C605: 47u, Capacitor_THT:CP_Radial_D6.3mm_P2.50mm, F.Cu at (232.4, 104.2)
- added C606: 1u 50V, Capacitor_THT:CP_Radial_D6.3mm_P2.50mm, F.Cu at (223.6, 112.3)
- added C607: 4u7, Capacitor_THT:CP_Radial_D6.3mm_P2.50mm, F.Cu at (221.1, 121.3)
- added C608: 100n, Capacitor_SMD:C_0805_2012Metric_Pad1.15x1.40mm_HandSolder, F.Cu at (235.8, 109.6)
- added C801: 100n, Capacitor_SMD:C_0805_2012Metric_Pad1.15x1.40mm_HandSolder, F.Cu at (196.8, 70.5)
- added C802: 100n, Capacitor_SMD:C_0805_2012Metric_Pad1.15x1.40mm_HandSolder, F.Cu at (195.8, 58.0)
- added C803: 100n, Capacitor_SMD:C_0805_2012Metric_Pad1.15x1.40mm_HandSolder, F.Cu at (191.8, 58.0)
- added C804: 100n, Capacitor_SMD:C_0805_2012Metric_Pad1.15x1.40mm_HandSolder, F.Cu at (185.8, 61.0)
- added C805: 100n, Capacitor_SMD:C_0805_2012Metric_Pad1.15x1.40mm_HandSolder, F.Cu at (199.8, 61.0)
- added C901: 100n, Capacitor_SMD:C_0805_2012Metric_Pad1.15x1.40mm_HandSolder, F.Cu at (159.5, 158.4)
- added C902: 6p, Capacitor_SMD:C_0805_2012Metric_Pad1.15x1.40mm_HandSolder, F.Cu at (179.2, 164.1)
- added C903: 6p, Capacitor_SMD:C_0805_2012Metric_Pad1.15x1.40mm_HandSolder, F.Cu at (165.8, 158.4)
- added D601: LED, LED_THT:LED_D3.0mm, F.Cu at (182.3, 140.7)
- added F601: 6A PTC, Fuse:Fuse_Bourns_MF-RG500, F.Cu at (210.7, 120.1)
- added FB401: 220R@100MHz, Inductor_SMD:L_0805_2012Metric_Pad1.15x1.40mm_HandSolder, F.Cu at (155.1, 87.8)
- added FB402: 220R@100MHz, Inductor_SMD:L_0805_2012Metric_Pad1.15x1.40mm_HandSolder, F.Cu at (155.8, 66.0)
- added FB403: 220R@100MHz, Inductor_SMD:L_0805_2012Metric_Pad1.15x1.40mm_HandSolder, F.Cu at (150.3, 87.8)
- added FB404: 220R@100MHz, Inductor_SMD:L_0805_2012Metric_Pad1.15x1.40mm_HandSolder, F.Cu at (155.8, 62.0)
- added FB405: 220R@100MHz, Inductor_SMD:L_0805_2012Metric_Pad1.15x1.40mm_HandSolder, F.Cu at (154.9, 84.8)
- added FB406: 220R@100MHz, Inductor_SMD:L_0805_2012Metric_Pad1.15x1.40mm_HandSolder, F.Cu at (143.2, 117.3)
- added FB407: 600R@100MHz, Inductor_SMD:L_0805_2012Metric_Pad1.15x1.40mm_HandSolder, F.Cu at (155.8, 58.0)
- added FB408: 220R@100MHz, Inductor_SMD:L_0805_2012Metric_Pad1.15x1.40mm_HandSolder, F.Cu at (150.1, 84.8)
- added FB409: 220R@100MHz, Inductor_SMD:L_0805_2012Metric_Pad1.15x1.40mm_HandSolder, F.Cu at (133.6, 88.3)
- added FB410: 220R@100MHz, Inductor_SMD:L_0805_2012Metric_Pad1.15x1.40mm_HandSolder, F.Cu at (151.3, 101.6)
- added FB411: 220R@100MHz, Inductor_SMD:L_0805_2012Metric_Pad1.15x1.40mm_HandSolder, F.Cu at (140.8, 85.8)
- added H101: MountingHole_Pad, MountingHole:MountingHole_4.3mm_M4_Pad_Via, F.Cu at (68.0, 41.3)
- added H102: MountingHole_Pad, MountingHole:MountingHole_4.3mm_M4_Pad_Via, F.Cu at (113.8, 41.3)
- added H103: MountingHole_Pad, MountingHole:MountingHole_4.3mm_M4_Pad_Via, F.Cu at (271.2, 64.2)
- added H104: MountingHole_Pad, MountingHole:MountingHole_4.3mm_M4_Pad_Via, F.Cu at (47.7, 196.3)
- added H105: MountingHole_Pad, MountingHole:MountingHole_4.3mm_M4_Pad_Via, F.Cu at (68.0, 196.3)
- added H106: MountingHole_Pad, MountingHole:MountingHole_4.3mm_M4_Pad_Via, F.Cu at (113.8, 196.3)
- added H107: MountingHole_Pad, MountingHole:MountingHole_4.3mm_M4_Pad_Via, F.Cu at (271.2, 196.3)
- added J1001: SD_Card, Connector_Card:SD_Kyocera_145638009211859+, F.Cu at (125.2, 168.3)
- added J101: Neotron-Expansion-Slot, Neotron-Common-Hardware:Neotron-Expansion-Slot, F.Cu at (115.2, 56.6)
- added J102: Neotron-Expansion-Slot, Neotron-Common-Hardware:Neotron-Expansion-Slot, F.Cu at (94.9, 56.6)
- added J103: Neotron-Expansion-Slot, Neotron-Common-Hardware:Neotron-Expansion-Slot, F.Cu at (72.2, 56.6)
- added J104: Neotron-Expansion-Slot, Neotron-Common-Hardware:Neotron-Expansion-Slot, F.Cu at (54.3, 56.6)
- added J201: DE15HD, Connector_Dsub:DSUB-15-HD_Female_Horizontal_P2.29x1.98mm_EdgePinOffset3.03mm_Housed_MountingHolesOffset4.94mm, F.Cu at (207.7, 38.7)
- added J301: RJ45 MagJack, Connector_RJ:RJ45_Amphenol_RJMG1BD3B8K1ANR, F.Cu at (157.8, 49.0)
- added J401: CD Audio In, Connector_PinHeader_2.54mm:PinHeader_1x04_P2.54mm_Vertical, F.Cu at (145.8, 56.0)
- added J402: AC'97 Audio Header, Connector_PinHeader_2.54mm:PinHeader_2x05_P2.54mm_Vertical, F.Cu at (138.8, 56.0)
- added J403: Line Out, Connector_PinHeader_2.54mm:PinHeader_1x04_P2.54mm_Vertical, F.Cu at (150.8, 56.0)
- added J501: USB Ports External, Neotron-Common-Hardware:CUI_UJ2-ADH-1-TH, F.Cu at (240.5, 43.9)
- added J502: USB Ports Internal, Neotron-Common-Hardware:USB_Header, F.Cu at (261.1, 64.2)
- added J601: Jack-DC, Connector_BarrelJack:BarrelJack_CUI_PJ-063AH_Horizontal, F.Cu at (252.2, 43.4)
- added J602: Conn_01x04, Connector_PinSocket_2.54mm:PinSocket_1x04_P2.54mm_Vertical, F.Cu at (178.4, 140.2)
- added J603: Double-mini-DIN-6, Neotron-Common-Hardware:Double_mini-DIN_6, F.Cu at (267.4, 42.1)
- added J801: Conn_02x05, Connector_IDC:IDC-Header_2x05_P2.54mm_Vertical, F.Cu at (197.8, 50.0)
- added J802: DB9_Male_MountingHoles, Connector_Dsub:DSUB-9_Male_Horizontal_P2.77x2.84mm_EdgePinOffset4.94mm_Housed_MountingHolesOffset7.48mm, F.Cu at (185.1, 39.8)
- added L601: 22u, Inductor_THT:L_Axial_L23.4mm_D12.7mm_P7.62mm_Vertical_Vishay_IHA-203, F.Cu at (240.8, 134.3)
- added LOGO101: OSHW Logo, Symbol:OSHW-Logo_11.4x12mm_SilkScreen, F.Cu at (258.6, 192.5)
- added LOGO102: Kicad Logo, Symbol:KiCad-Logo2_12mm_SilkScreen, F.Cu at (235.7, 189.9)
- added LOGO103: Neotron Logo, Neotron-Common-Hardware:logo, F.Cu at (188.7, 189.9)
- added R201: 75, Resistor_SMD:R_0805_2012Metric_Pad1.15x1.40mm_HandSolder, F.Cu at (253.7, 76.7)
- added R202: 75, Resistor_SMD:R_0805_2012Metric_Pad1.15x1.40mm_HandSolder, F.Cu at (248.9, 79.6)
- added R203: 75, Resistor_SMD:R_0805_2012Metric_Pad1.15x1.40mm_HandSolder, F.Cu at (245.7, 82.6)
- added R204: 10k, Resistor_SMD:R_0805_2012Metric_Pad1.15x1.40mm_HandSolder, F.Cu at (240.9, 87.5)
- added R205: 10k, Resistor_SMD:R_0805_2012Metric_Pad1.15x1.40mm_HandSolder, F.Cu at (248.9, 76.7)
- added R206: 10k, Resistor_SMD:R_0805_2012Metric_Pad1.15x1.40mm_HandSolder, F.Cu at (244.2, 79.6)
- added R207: 1k5, Resistor_SMD:R_0805_2012Metric_Pad1.15x1.40mm_HandSolder, F.Cu at (240.9, 84.5)
- added R208: 1k5, Resistor_SMD:R_0805_2012Metric_Pad1.15x1.40mm_HandSolder, F.Cu at (236.2, 87.5)
- added R209: DNF, Resistor_SMD:R_0805_2012Metric_Pad1.15x1.40mm_HandSolder, F.Cu at (244.2, 76.7)
- added R301: 100k, Resistor_SMD:R_0805_2012Metric_Pad1.15x1.40mm_HandSolder, F.Cu at (177.7, 84.5)
- added R302: 49R9 1%, Resistor_SMD:R_0805_2012Metric_Pad1.15x1.40mm_HandSolder, F.Cu at (169.1, 66.6)
- added R303: 49R9 1%, Resistor_SMD:R_0805_2012Metric_Pad1.15x1.40mm_HandSolder, F.Cu at (166.2, 61.9)
- added R304: 49R9 1%, Resistor_SMD:R_0805_2012Metric_Pad1.15x1.40mm_HandSolder, F.Cu at (172.1, 67.0)
- added R305: 49R9 1%, Resistor_SMD:R_0805_2012Metric_Pad1.15x1.40mm_HandSolder, F.Cu at (175.0, 70.3)
- added R306: 12k4 1%, Resistor_SMD:R_0805_2012Metric_Pad1.15x1.40mm_HandSolder, F.Cu at (169.1, 61.9)
- added R307: 1M, Resistor_SMD:R_0805_2012Metric_Pad1.15x1.40mm_HandSolder, F.Cu at (178.0, 70.3)
- added R308: 10, Resistor_SMD:R_0805_2012Metric_Pad1.15x1.40mm_HandSolder, F.Cu at (172.1, 62.3)
- added R309: 10, Resistor_SMD:R_0805_2012Metric_Pad1.15x1.40mm_HandSolder, F.Cu at (175.0, 65.5)
- added R310: 180, Resistor_SMD:R_0805_2012Metric_Pad1.15x1.40mm_HandSolder, F.Cu at (178.0, 65.5)
- added R311: 180, Resistor_SMD:R_0805_2012Metric_Pad1.15x1.40mm_HandSolder, F.Cu at (172.1, 57.5)
- added R312: DNF, Resistor_SMD:R_0805_2012Metric_Pad1.15x1.40mm_HandSolder, F.Cu at (175.0, 60.8)
- added R401: 2R2, Resistor_SMD:R_0805_2012Metric_Pad1.15x1.40mm_HandSolder, F.Cu at (155.8, 94.0)
- added R402: 2R2, Resistor_SMD:R_0805_2012Metric_Pad1.15x1.40mm_HandSolder, F.Cu at (129.2, 110.2)
- added R403: 2R2, Resistor_SMD:R_0805_2012Metric_Pad1.15x1.40mm_HandSolder, F.Cu at (129.2, 106.2)
- added R404: 100, Resistor_SMD:R_0805_2012Metric_Pad1.15x1.40mm_HandSolder, F.Cu at (115.9, 94.0)
- added R405: 100, Resistor_SMD:R_0805_2012Metric_Pad1.15x1.40mm_HandSolder, F.Cu at (115.9, 122.4)
- added R406: 47k, Resistor_SMD:R_0805_2012Metric_Pad1.15x1.40mm_HandSolder, F.Cu at (142.5, 98.1)
- added R407: 47k, Resistor_SMD:R_0805_2012Metric_Pad1.15x1.40mm_HandSolder, F.Cu at (115.9, 118.3)
- added R408: 4k7, Resistor_SMD:R_0805_2012Metric_Pad1.15x1.40mm_HandSolder, F.Cu at (129.2, 102.1)
- added R409: 47k, Resistor_SMD:R_0805_2012Metric_Pad1.15x1.40mm_HandSolder, F.Cu at (115.9, 114.3)
- added R410: 47k, Resistor_SMD:R_0805_2012Metric_Pad1.15x1.40mm_HandSolder, F.Cu at (142.5, 94.0)
- added R411: 2k2, Resistor_SMD:R_0805_2012Metric_Pad1.15x1.40mm_HandSolder, F.Cu at (115.9, 110.2)
- added R412: 4k7, Resistor_SMD:R_0805_2012Metric_Pad1.15x1.40mm_HandSolder, F.Cu at (115.9, 106.2)
- added R413: 4k7, Resistor_SMD:R_0805_2012Metric_Pad1.15x1.40mm_HandSolder, F.Cu at (129.2, 98.1)
- added R414: 4k7, Resistor_SMD:R_0805_2012Metric_Pad1.15x1.40mm_HandSolder, F.Cu at (115.9, 102.1)
- added R415: 4k7, Resistor_SMD:R_0805_2012Metric_Pad1.15x1.40mm_HandSolder, F.Cu at (129.2, 94.0)
- added R416: 10k, Resistor_SMD:R_0805_2012Metric_Pad1.15x1.40mm_HandSolder, F.Cu at (115.9, 98.1)
- added R501: 2k7 1%, Resistor_SMD:R_0805_2012Metric_Pad1.15x1.40mm_HandSolder, F.Cu at (228.4, 76.7)
- added R502: 10k, Resistor_SMD:R_0805_2012Metric_Pad1.15x1.40mm_HandSolder, F.Cu at (260.3, 97.5)
- added R503: 10k, Resistor_SMD:R_0805_2012Metric_Pad1.15x1.40mm_HandSolder, F.Cu at (220.4, 87.5)
- added R504: 10k, Resistor_SMD:R_0805_2012Metric_Pad1.15x1.40mm_HandSolder, F.Cu at (228.4, 79.6)
- added R506: 10k, Resistor_SMD:R_0805_2012Metric_Pad1.15x1.40mm_HandSolder, F.Cu at (260.3, 94.6)
- added R507: 10k, Resistor_SMD:R_0805_2012Metric_Pad1.15x1.40mm_HandSolder, F.Cu at (130.5, 78.2)
- added R508: 10k, Resistor_SMD:R_0805_2012Metric_Pad1.15x1.40mm_HandSolder, F.Cu at (131.6, 65.5)
- added R509: 10k, Resistor_SMD:R_0805_2012Metric_Pad1.15x1.40mm_HandSolder, F.Cu at (130.5, 83.2)
- added R601: 100k, Resistor_SMD:R_0805_2012Metric_Pad1.15x1.40mm_HandSolder, F.Cu at (217.9, 126.7)
- added R602: 100k, Resistor_SMD:R_0805_2012Metric_Pad1.15x1.40mm_HandSolder, F.Cu at (178.4, 151.6)
- added R603: 100k, Resistor_SMD:R_0805_2012Metric_Pad1.15x1.40mm_HandSolder, F.Cu at (183.1, 144.9)
- added R604: 1k, Resistor_SMD:R_0805_2012Metric_Pad1.15x1.40mm_HandSolder, F.Cu at (187.8, 144.9)
- added R605: 33k, Resistor_SMD:R_0805_2012Metric_Pad1.15x1.40mm_HandSolder, F.Cu at (183.1, 147.9)
- added R606: 100k, Resistor_SMD:R_0805_2012Metric_Pad1.15x1.40mm_HandSolder, F.Cu at (228.7, 117.7)
- added R607: 100k, Resistor_SMD:R_0805_2012Metric_Pad1.15x1.40mm_HandSolder, F.Cu at (183.2, 150.8)
- added R608: 100k, Resistor_SMD:R_0805_2012Metric_Pad1.15x1.40mm_HandSolder, F.Cu at (244.6, 101.8)
- added R801: DNF, Resistor_SMD:R_0805_2012Metric_Pad1.15x1.40mm_HandSolder, F.Cu at (115.9, 136.9)
- added RN1001: 8x10k, Resistor_THT:R_Array_SIP9, F.Cu at (132.8, 148.0)
- added RN601: 2k7 x 4, Resistor_THT:R_Array_SIP5, F.Cu at (254.5, 102.8)
- added SW601: SW_DIP_x01, Connector_PinHeader_2.54mm:PinHeader_1x02_P2.54mm_Vertical, F.Cu at (239.9, 102.6)
- added SW602: SW_DIP_x01, Connector_PinHeader_2.54mm:PinHeader_1x02_P2.54mm_Vertical, F.Cu at (231.1, 110.7)
- added TP601: Reset, TestPoint:TestPoint_THTPad_2.0x2.0mm_Drill1.0mm, F.Cu at (217.6, 130.2)
- added U101: Neotron-CPU, Neotron-Common-Hardware:Neotron_CPU_Socket, F.Cu at (220.4, 163.3)
- added U201: THS7316, Package_SO:SOIC-8_3.9x4.9mm_P1.27mm, F.Cu at (232.9, 53.5)
- added U202: TPD7S019, Package_SO:SSOP-16_3.9x4.9mm_P0.635mm, F.Cu at (221.2, 53.3)
- added U301: ENC424J600, Package_QFP:TQFP-44_10x10mm_P0.8mm, F.Cu at (187.8, 82.0)
- added U401: TLV320AIC23BPW, Package_SO:TSSOP-28_4.4x9.7mm_P0.65mm, F.Cu at (148.8, 74.0)
- added U402: STX-4335-5BGP-S1, Neotron-Common-Hardware:STX-4335-5BGP-S1, F.Cu at (135.8, 39.0)
- added U501: AP2501, Package_SO:SO-8_3.9x4.9mm_P1.27mm, F.Cu at (252.4, 94.0)
- added U502: MIC2005A-2YM5, Package_TO_SOT_SMD:SOT-23-5_HandSoldering, F.Cu at (247.1, 52.5)
- added U503: MIC2005A-2YM5, Package_TO_SOT_SMD:SOT-23-5_HandSoldering, F.Cu at (253.6, 52.5)
- added U504: XR22404CG28, Package_SO:SSOP-28_3.9x9.9mm_P0.635mm, F.Cu at (249.7, 61.7)
- added U505: MIC2005A-2YM5, Package_TO_SOT_SMD:SOT-23-5_HandSoldering, F.Cu at (257.2, 62.9)
- added U506: MIC2005A-2YM5, Package_TO_SOT_SMD:SOT-23-5_HandSoldering, F.Cu at (257.2, 59.1)
- added U601: 5V DC-DC Module, Connector_PinSocket_2.54mm:PinSocket_1x12_P2.54mm_Vertical, F.Cu at (270.7, 80.5)
- added U602: 3v3 LDO, Package_TO_SOT_SMD:TO-252-3_TabPin2, F.Cu at (201.4, 125.5)
- added U603: MAX1615, Package_TO_SOT_SMD:SOT-23-5, F.Cu at (203.7, 133.1)
- added U604: MKE04P24M48SF0, Package_SO:SOIC-20W_7.5x12.8mm_P1.27mm, F.Cu at (169.6, 145.1)
- added U801: ST3232CDR, Package_SO:SO-16_5.3x10.2mm_P1.27mm, F.Cu at (192.8, 64.2)
- added U901: MCP7940, Package_SO:SOIC-8_3.9x4.9mm_P1.27mm, F.Cu at (174.5, 162.3)
- added Y301: 25M, Crystal:Crystal_HC49-4H_Vertical, F.Cu at (165.1, 82.8)
- added Y401: 12M, Crystal:Crystal_HC49-4H_Vertical, F.Cu at (131.8, 115.6)
- added Y501: 12M, Crystal:Crystal_HC49-4H_Vertical, F.Cu at (242.0, 64.2)
- added Y901: 32,768 Hz, Crystal:Crystal_C26-LF_D2.1mm_L6.5mm_Horizontal, F.Cu at (161.5, 165.1)
Routing:
- net Net-(R507-Pad2): track 0.00 -> 1.24 mm, vias 0 -> 1
- net Net-(R509-Pad2): track 0.00 -> 1.24 mm, vias 0 -> 1
- net /USB/USB_3V3: track 0.00 -> 1.24 mm, vias 0 -> 1
- added copper zone on In2.Cu, net +3V3
- added copper zone on In1.Cu, net GND
Other:
- board outline added: 243.8 x 170.2 mm
- copper layers 2 -> 4
- board text added: "2x USB Type-A"
- board text added: "Cards are at 0.800" centres. NOTE: They are the "PCI" way around, i.e. components to the left, NOT the "ISA" way around. This is so a single slot fits on an ITX board."
- board text added: "DC In"
- board text added: "Dual PS/2"
- board text added: "Ethernet"
- board text added: "PCB Version: [Uncontrolled]"
- board text added: "RS-232"
- board text added: "Slot 1"
- board text added: "Stereo Audio In/Out/Mic"
- board text added: "Super VGA"
- board text added: "https://neotron-compute.github.io"

Commit message: Updated common to 0.4.0 and added some part numbers.
Parts:
- added R301: 24k 0.5%, Resistor_SMD:R_0805_2012Metric_Pad1.15x1.40mm_HandSolder, F.Cu at (66.8, 108.7)
- added R302: 24k 0.5%, Resistor_SMD:R_0805_2012Metric_Pad1.15x1.40mm_HandSolder, F.Cu at (57.3, 108.7)
- added R303: 24k 0.5%, Resistor_SMD:R_0805_2012Metric_Pad1.15x1.40mm_HandSolder, F.Cu at (57.3, 117.5)
- added R304: 24k 0.5%, Resistor_SMD:R_0805_2012Metric_Pad1.15x1.40mm_HandSolder, F.Cu at (62.0, 114.5)
- added R305: 24k 0.5%, Resistor_SMD:R_0805_2012Metric_Pad1.15x1.40mm_HandSolder, F.Cu at (66.8, 111.6)
- added R306: 24k 0.5%, Resistor_SMD:R_0805_2012Metric_Pad1.15x1.40mm_HandSolder, F.Cu at (71.5, 108.7)
- added R307: 12k 0.5%, Resistor_SMD:R_0805_2012Metric_Pad1.15x1.40mm_HandSolder, F.Cu at (71.5, 111.6)
- added R308: 12k 0.5%, Resistor_SMD:R_0805_2012Metric_Pad1.15x1.40mm_HandSolder, F.Cu at (66.8, 114.5)
- added R309: 12k 0.5%, Resistor_SMD:R_0805_2012Metric_Pad1.15x1.40mm_HandSolder, F.Cu at (62.0, 111.6)
- added R310: 12k 0.5%, Resistor_SMD:R_0805_2012Metric_Pad1.15x1.40mm_HandSolder, F.Cu at (62.0, 117.5)
- added R311: 12k 0.5%, Resistor_SMD:R_0805_2012Metric_Pad1.15x1.40mm_HandSolder, F.Cu at (57.3, 114.5)
- added R312: 24k 0.5%, Resistor_SMD:R_0805_2012Metric_Pad1.15x1.40mm_HandSolder, F.Cu at (62.0, 108.7)
- added R313: 3300, Resistor_SMD:R_0805_2012Metric_Pad1.15x1.40mm_HandSolder, F.Cu at (57.3, 111.6)
- added R401: 24k 0.5%, Resistor_SMD:R_0805_2012Metric_Pad1.15x1.40mm_HandSolder, F.Cu at (57.3, 126.9)
- added R402: 24k 0.5%, Resistor_SMD:R_0805_2012Metric_Pad1.15x1.40mm_HandSolder, F.Cu at (62.0, 123.9)
- added R403: 24k 0.5%, Resistor_SMD:R_0805_2012Metric_Pad1.15x1.40mm_HandSolder, F.Cu at (57.3, 132.8)
- added R404: 24k 0.5%, Resistor_SMD:R_0805_2012Metric_Pad1.15x1.40mm_HandSolder, F.Cu at (57.3, 123.9)
- added R405: 24k 0.5%, Resistor_SMD:R_0805_2012Metric_Pad1.15x1.40mm_HandSolder, F.Cu at (62.0, 129.8)
- added R406: 24k 0.5%, Resistor_SMD:R_0805_2012Metric_Pad1.15x1.40mm_HandSolder, F.Cu at (66.8, 126.9)
- added R407: 12k 0.5%, Resistor_SMD:R_0805_2012Metric_Pad1.15x1.40mm_HandSolder, F.Cu at (71.5, 123.9)
- added R408: 12k 0.5%, Resistor_SMD:R_0805_2012Metric_Pad1.15x1.40mm_HandSolder, F.Cu at (62.0, 132.8)
- added R409: 12k 0.5%, Resistor_SMD:R_0805_2012Metric_Pad1.15x1.40mm_HandSolder, F.Cu at (66.8, 129.8)
- added R410: 12k 0.5%, Resistor_SMD:R_0805_2012Metric_Pad1.15x1.40mm_HandSolder, F.Cu at (66.8, 123.9)
- added R411: 12k 0.5%, Resistor_SMD:R_0805_2012Metric_Pad1.15x1.40mm_HandSolder, F.Cu at (71.5, 126.9)
- added R412: 24k 0.5%, Resistor_SMD:R_0805_2012Metric_Pad1.15x1.40mm_HandSolder, F.Cu at (62.0, 126.9)
- added R413: 3300, Resistor_SMD:R_0805_2012Metric_Pad1.15x1.40mm_HandSolder, F.Cu at (57.3, 129.8)
- added R501: 24k 0.5%, Resistor_SMD:R_0805_2012Metric_Pad1.15x1.40mm_HandSolder, F.Cu at (96.3, 111.6)
- added R502: 24k 0.5%, Resistor_SMD:R_0805_2012Metric_Pad1.15x1.40mm_HandSolder, F.Cu at (91.5, 114.5)
- added R503: 24k 0.5%, Resistor_SMD:R_0805_2012Metric_Pad1.15x1.40mm_HandSolder, F.Cu at (86.8, 117.5)
- added R504: 24k 0.5%, Resistor_SMD:R_0805_2012Metric_Pad1.15x1.40mm_HandSolder, F.Cu at (82.0, 108.7)
- added R505: 24k 0.5%, Resistor_SMD:R_0805_2012Metric_Pad1.15x1.40mm_HandSolder, F.Cu at (82.0, 111.6)
- added R506: 24k 0.5%, Resistor_SMD:R_0805_2012Metric_Pad1.15x1.40mm_HandSolder, F.Cu at (86.8, 108.7)
- added R507: 12k 0.5%, Resistor_SMD:R_0805_2012Metric_Pad1.15x1.40mm_HandSolder, F.Cu at (82.0, 114.5)
- added R508: 12k 0.5%, Resistor_SMD:R_0805_2012Metric_Pad1.15x1.40mm_HandSolder, F.Cu at (86.8, 111.6)
- added R509: 12k 0.5%, Resistor_SMD:R_0805_2012Metric_Pad1.15x1.40mm_HandSolder, F.Cu at (91.5, 108.7)
- added R510: 12k 0.5%, Resistor_SMD:R_0805_2012Metric_Pad1.15x1.40mm_HandSolder, F.Cu at (82.0, 117.5)
- added R511: 12k 0.5%, Resistor_SMD:R_0805_2012Metric_Pad1.15x1.40mm_HandSolder, F.Cu at (86.8, 114.5)
- added R512: 24k 0.5%, Resistor_SMD:R_0805_2012Metric_Pad1.15x1.40mm_HandSolder, F.Cu at (91.5, 111.6)
- added R513: 3300, Resistor_SMD:R_0805_2012Metric_Pad1.15x1.40mm_HandSolder, F.Cu at (96.3, 108.7)
- added TP101: TestPoint, TestPoint:TestPoint_THTPad_D2.0mm_Drill1.0mm, F.Cu at (89.8, 124.5)
- added TP102: TestPoint, TestPoint:TestPoint_THTPad_D2.0mm_Drill1.0mm, F.Cu at (85.8, 128.5)
- added TP103: TestPoint, TestPoint:TestPoint_THTPad_D2.0mm_Drill1.0mm, F.Cu at (85.8, 124.5)
- added TP104: TestPoint, TestPoint:TestPoint_THTPad_D2.0mm_Drill1.0mm, F.Cu at (81.7, 128.5)
- added TP105: TestPoint, TestPoint:TestPoint_THTPad_D2.0mm_Drill1.0mm, F.Cu at (81.7, 124.5)
- C1006: renamed from C504; footprint Capacitor_THT:CP_Radial_D6.3mm_P2.50mm -> Capacitor_THT:CP_Radial_D8.0mm_P3.50mm
- C1007: renamed from C505; footprint Capacitor_THT:CP_Radial_D6.3mm_P2.50mm -> Capacitor_THT:CP_Radial_D8.0mm_P3.50mm
- C1010: renamed from C509; footprint Capacitor_THT:CP_Radial_D6.3mm_P2.50mm -> Capacitor_THT:CP_Radial_D8.0mm_P3.50mm
- C1011: renamed from C510; footprint Capacitor_THT:CP_Radial_D6.3mm_P2.50mm -> Capacitor_THT:CP_Radial_D8.0mm_P3.50mm
- C901: renamed from C601; footprint Capacitor_THT:CP_Radial_D6.3mm_P2.50mm -> Capacitor_THT:CP_Radial_D8.0mm_P3.50mm
- C902: renamed from C602; footprint Capacitor_THT:CP_Radial_D6.3mm_P2.50mm -> Capacitor_THT:CP_Radial_D8.0mm_P3.50mm
- J802: footprint Connector_Dsub:DSUB-9_Male_Horizontal_P2.77x2.84mm_EdgePinOffset4.94mm_Housed_MountingHolesOffset7.48mm -> Connector_Dsub:DSUB-9_Male_Horizontal_P2.77x2.84mm_EdgePinOffset7.70mm_Housed_MountingHolesOffset9.12mm
- renumbered BT901 to BT1201, C501 to C1001, C508 to C1002, C511 to C1003, C502 to C1004, C503 to C1005, C506 to C1008, C507 to C1009, C310 to C1101, C311 to C1102, C309 to C1103, C312 to C1104, C308 to C1105, C301 to C1106, C302 to C1107, C303 to C1108, C304 to C1109, C305 to C1110, C306 to C1111, C307 to C1112, C901 to C1201, C902 to C1202, C903 to C1203, C412 to C601, C413 to C602, C407 to C603, C411 to C604, C418 to C605, C419 to C606, C424 to C607, C427 to C608, C431 to C609, C435 to C610, C402 to C611, C406 to C612, C408 to C613, C420 to C614, C421 to C615, C426 to C616, C428 to C617, C432 to C618, C437 to C619, C422 to C620, C423 to C621, C430 to C622, C433 to C623, C436 to C624, C438 to C625, C415 to C626, C416 to C627, C401 to C628, C405 to C629, C425 to C630, C429 to C631, C434 to C632, C403 to C633, C409 to C634, C414 to C635, C417 to C636, C404 to C637, C410 to C638, C1001 to C701, C1002 to C702, C802 to C801, C803 to C802, C805 to C803, C801 to C805, C603 to C903, C604 to C904, C605 to C905, C606 to C906, C607 to C907, C608 to C908, D601 to D901, F601 to F901, FB405 to FB601, FB409 to FB602, FB406 to FB603, FB410 to FB604, FB408 to FB605, FB411 to FB606, FB407 to FB607, FB401 to FB608, FB403 to FB609, FB402 to FB610, FB404 to FB611, J501 to J1001, J502 to J1002, J301 to J1101, J403 to J601, J402 to J602, J401 to J603, J1001 to J701, J601 to J901, J602 to J902, J603 to J903, L601 to L901, LOGO103 to LOGO101, LOGO101 to LOGO103, R502 to R1001, R501 to R1002, R503 to R1003, R504 to R1004, R507 to R1005, R508 to R1006, R509 to R1007, R506 to R1008, R302 to R1101, R308 to R1102, R303 to R1103, R304 to R1104, R301 to R1105, R309 to R1106, R305 to R1107, R311 to R1108, R310 to R1109, R312 to R1110, R307 to R1111, R306 to R1112, R209 to R207, R207 to R208, R208 to R209, R404 to R601, R405 to R602, R406 to R603, R409 to R604, R407 to R605, R410 to R606, R414 to R607, R415 to R608, R408 to R609, R413 to R610, R411 to R611, R412 to R612, R416 to R613, R401 to R614, R403 to R615, R402 to R616, R601 to R901, R602 to R902, R603 to R903, R604 to R904, R606 to R905, R605 to R906, R608 to R907, R607 to R908, RN1001 to RN701, RN601 to RN901, SW601 to SW901, SW602 to SW902, TP601 to TP901, U501 to U1001, U502 to U1002, U503 to U1003, U504 to U1004, U505 to U1005, U506 to U1006, U301 to U1101, U901 to U1201, U401 to U601, U402 to U602, U601 to U901, U602 to U902, U603 to U903, U604 to U904, Y501 to Y1001, Y301 to Y1101, Y901 to Y1201, Y401 to Y601
Connections:
- J101 pad 1: (no net) -> /SPI_COPI
- J101 pad 10: (no net) -> /I2C_SDA
- J101 pad 14: (no net) -> /~RESET
- J101 pad 3: (no net) -> /SPI_CIPO
- J101 pad 5: (no net) -> /SPI_CLK
- J101 pad 7: (no net) -> /~CS0
- J101 pad 8: (no net) -> /~IRQ0
- J101 pad 9: (no net) -> /I2C_SCL
- J102 pad 1: (no net) -> /SPI_COPI
- J102 pad 10: (no net) -> /I2C_SDA
- J102 pad 14: (no net) -> /~RESET
- J102 pad 3: (no net) -> /SPI_CIPO
- J102 pad 5: (no net) -> /SPI_CLK
- J102 pad 7: (no net) -> /~CS1
- J102 pad 8: (no net) -> /~IRQ1
- J102 pad 9: (no net) -> /I2C_SCL
- J103 pad 1: (no net) -> /SPI_COPI
- J103 pad 10: (no net) -> /I2C_SDA
- J103 pad 14: (no net) -> /~RESET
- J103 pad 3: (no net) -> /SPI_CIPO
- J103 pad 5: (no net) -> /SPI_CLK
- J103 pad 7: (no net) -> /~CS2
- J103 pad 8: (no net) -> /~IRQ2
- J103 pad 9: (no net) -> /I2C_SCL
- J104 pad 1: (no net) -> /SPI_COPI
- J104 pad 10: (no net) -> /I2C_SDA
- J104 pad 14: (no net) -> /~RESET
- J104 pad 3: (no net) -> /SPI_CIPO
- J104 pad 5: (no net) -> /SPI_CLK
- J104 pad 7: (no net) -> /~CS3
- J104 pad 8: (no net) -> /~IRQ3
- J104 pad 9: (no net) -> /I2C_SCL
- R1105 pad 2: /Ethernet/~IRQ -> /~IRQ4
- U1004 pad 15: (no net) -> /USB/USBD-
- U1004 pad 16: (no net) -> /USB/USBD+
- U101 pad 1.1: (no net) -> /R5
- U101 pad 1.10: (no net) -> /G2
- U101 pad 1.11: (no net) -> /G1
- U101 pad 1.12: (no net) -> /G0
- U101 pad 1.13: (no net) -> /B5
- U101 pad 1.14: (no net) -> /B4
- U101 pad 1.15: (no net) -> /B3
- U101 pad 1.16: (no net) -> /B2
- U101 pad 1.17: (no net) -> /B1
- U101 pad 1.18: (no net) -> /B0
- U101 pad 1.19: (no net) -> /Video/HSYNC
- U101 pad 1.2: (no net) -> /R4
- U101 pad 1.20: (no net) -> /Video/VSYNC
- U101 pad 1.3: (no net) -> /R3
- U101 pad 1.4: (no net) -> /R2
- U101 pad 1.5: (no net) -> /R1
- U101 pad 1.6: (no net) -> /R0
- U101 pad 1.7: (no net) -> /G5
- U101 pad 1.8: (no net) -> /G4
- U101 pad 1.9: (no net) -> /G3
- U101 pad 2.1: (no net) -> /Video/DDC_SDA
- U101 pad 2.13: (no net) -> /Audio/AUDIO_BIT_CLK_TO_CODEC
- U101 pad 2.14: (no net) -> /Audio/AUDIO_DAT_TO_CODEC
- U101 pad 2.15: (no net) -> /Audio/AUDIO_LR_TO_CODEC
- U101 pad 2.16: (no net) -> /Audio/AUDIO_DAT_FROM_CODEC
- U101 pad 2.17: (no net) -> /Audio/AUDIO_LR_FROM_CODEC
- U101 pad 2.18: (no net) -> /USB/~ENABLE
- U101 pad 2.19: (no net) -> /USB/USBD-
- U101 pad 2.2: (no net) -> /Video/DDC_SCL
- U101 pad 2.20: (no net) -> /USB/USBD+
- U101 pad 2.3: (no net) -> /Serial/RS232_RX_TO_MCU
- U101 pad 2.4: (no net) -> /Serial/RS232_TX_FROM_MCU
- U101 pad 3.1: (no net) -> /I2C_SDA
- U101 pad 3.13: (no net) -> /~CS7
- U101 pad 3.14: (no net) -> /~CS6
- U101 pad 3.15: (no net) -> /~CS5
- U101 pad 3.16: (no net) -> /~CS4
- U101 pad 3.17: (no net) -> /~CS3
- U101 pad 3.18: (no net) -> /~CS2
- U101 pad 3.19: (no net) -> /~CS1
- U101 pad 3.2: (no net) -> /I2C_SCL
- U101 pad 3.20: (no net) -> /~CS0
- U101 pad 3.3: (no net) -> /Serial/RS232_CTS_TO_MCU
- U101 pad 3.4: (no net) -> /Serial/RS232_RTS_FROM_MCU
- U101 pad 4.1: (no net) -> /SD Card/~CARD_DETECT
- U101 pad 4.10: (no net) -> /SPI_CIPO
- U101 pad 4.11: (no net) -> /SPI_CLK
- U101 pad 4.12: (no net) -> /~RESET
- U101 pad 4.13: (no net) -> /~IRQ7
- U101 pad 4.14: (no net) -> /~IRQ6
- U101 pad 4.15: (no net) -> /~IRQ5
- U101 pad 4.16: (no net) -> /~IRQ4
- U101 pad 4.17: (no net) -> /~IRQ3
- U101 pad 4.18: (no net) -> /~IRQ2
- U101 pad 4.19: (no net) -> /~IRQ1
- U101 pad 4.2: (no net) -> /SD Card/~WRITE_PROTECT
- U101 pad 4.20: (no net) -> /~IRQ0
- U101 pad 4.3: (no net) -> /SD Card/DAT2
- U101 pad 4.4: (no net) -> /SD Card/DAT3
- U101 pad 4.5: (no net) -> /SD Card/CMD
- U101 pad 4.6: (no net) -> /SD Card/CLK
- U101 pad 4.7: (no net) -> /SD Card/DAT0
- U101 pad 4.8: (no net) -> /SD Card/DAT1
- U101 pad 4.9: (no net) -> /SPI_COPI
- U1101 pad 24: /Ethernet/~IRQ -> /~IRQ4
- U1101 pad 34: (no net) -> /~CS4
- U1101 pad 35: (no net) -> /SPI_CIPO
- U1101 pad 36: (no net) -> /SPI_COPI
- U1101 pad 37: (no net) -> /SPI_CLK
- U1201 pad 5: (no net) -> /I2C_SDA
- U1201 pad 6: (no net) -> /I2C_SCL
- U202 pad 10: (no net) -> /Video/DDC_SDA
- U202 pad 11: (no net) -> /Video/DDC_SCL
- U202 pad 13: (no net) -> /Video/VSYNC
- U202 pad 15: (no net) -> /Video/HSYNC
- U601 pad 23: (no net) -> /I2C_SDA
- U601 pad 24: (no net) -> /I2C_SCL
- U601 pad 3: (no net) -> /Audio/AUDIO_BIT_CLK_TO_CODEC
- U601 pad 4: (no net) -> /Audio/AUDIO_DAT_TO_CODEC
- U601 pad 5: (no net) -> /Audio/AUDIO_LR_TO_CODEC
- U601 pad 6: (no net) -> /Audio/AUDIO_DAT_FROM_CODEC
- U601 pad 7: (no net) -> /Audio/AUDIO_LR_FROM_CODEC
- U801 pad 10: (no net) -> /Serial/RS232_RTS_FROM_MCU
- U801 pad 11: (no net) -> /Serial/RS232_TX_FROM_MCU
- U801 pad 12: (no net) -> /Serial/RS232_RX_TO_MCU
- U801 pad 9: (no net) -> /Serial/RS232_CTS_TO_MCU
- U904 pad 14: (no net) -> /~IRQ7
- U904 pad 17: (no net) -> /I2C_SCL
- U904 pad 18: (no net) -> /I2C_SDA
- U904 pad 7: (no net) -> /~RESET

Commit message: Working on PSU layout.
Parts:
- moved U201 399.2 mm to (-144.3, 184.3)
- moved U202 399.2 mm to (-156.0, 184.1)
- moved C701 322.7 mm to (-65.3, 178.5)
- moved C801 288.3 mm to (-91.2, 84.7)
- moved C802 288.3 mm to (-95.2, 84.7)
- moved C803 288.3 mm to (-87.3, 87.7)
- moved C804 288.3 mm to (-101.3, 87.7)
- moved R1108 288.3 mm to (-115.0, 84.2)
- moved R1110 288.3 mm to (-112.0, 87.4)
- moved C608 267.7 mm to (-150.8, 152.6)
- moved C612 267.7 mm to (-86.9, 124.5)
- moved C613 267.7 mm to (-116.9, 152.1)
- moved C617 267.7 mm to (-150.8, 149.0)
- moved C619 267.7 mm to (-94.6, 135.9)
- moved C622 267.7 mm to (-94.6, 132.3)
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Connections:
- RN901 pad 4: /Power Supply/PS2_CLK1 -> /Power Supply/PS2_DAT1
- RN901 pad 5: /Power Supply/PS2_DAT1 -> /Power Supply/PS2_CLK1
Routing:
- net +5V: track 0.00 -> 188.5 mm
- net /Power Supply/PS2_DAT1: track 0.00 -> 144.9 mm, vias 0 -> 1
- net /Power Supply/PS2_CLK1: track 0.00 -> 137.1 mm, vias 0 -> 1
- net /Power Supply/PS2_DAT0: track 0.00 -> 86.9 mm
- net /Power Supply/PS2_CLK0: track 0.00 -> 75.1 mm
- net /I2C_SCL: track 0.00 -> 64.3 mm
- net /I2C_SDA: track 0.00 -> 64.0 mm
- net /SPI_COPI: track 0.00 -> 63.7 mm
- net /~RESET: track 0.00 -> 63.7 mm
- net /SPI_CLK: track 0.00 -> 63.7 mm
- net /SPI_CIPO: track 0.00 -> 63.7 mm
- net +3V3: track 0.11 -> 57.7 mm, vias 0 -> 11
- net +5VP: track 0.00 -> 55.9 mm
- net Net-(C902-Pad1): track 0.00 -> 50.1 mm
- net /Power Supply/DC_ON: track 0.00 -> 36.5 mm, vias 0 -> 1
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- added copper zone on Vcc.Cu, net +3V3
- added copper zone on Gnd.Cu, net GND
- removed copper zone on In2.Cu, net +3V3
- removed copper zone on In1.Cu, net GND
Other:
- net class DC_In added: clearance 0.127, trace_width 2, via_dia 0.8, via_drill 0.4
- net class Default: clearance 0.2 -> 0.127; trace_width 0.25 -> 0.2
- net class Power added: clearance 0.127, trace_width 0.5, via_dia 0.8, via_drill 0.4
- net class USB added: clearance 0.2, trace_width 0.45, via_dia 0.8, via_drill 0.4
- rule trace_clearance: 0.2 -> 0.127
- rule trace_min: 0.2 -> 0.0889
- rule via_min_drill: 0.3 -> 0.2
- rule via_min_size: 0.4 -> 0.45
- board text added: "Baseboard 100, [Uncontrolled]"
- board text added: "JLCJLCJLCJLC"
- board text added: "Power Supply"
- board text removed: "PCB Version: [Uncontrolled]"
- board text removed: "https://neotron-compute.github.io"

Commit message: Working on laying out USB hub.
Parts:
- moved U202 395.9 mm to (214.2, 43.8), turned to 0 degrees
- moved U201 373.6 mm to (201.8, 43.7), turned to 0 degrees
- moved R209 248.0 mm to (220.7, 42.2), turned to 180 degrees
- moved C203 243.1 mm to (228.3, -0.37)
- moved C206 243.1 mm to (211.2, -0.87)
- moved R207 243.1 mm to (218.8, -3.32)
- moved C201 243.1 mm to (225.0, 5.53)
- moved C202 243.1 mm to (210.8, 4.53)
- moved C204 243.1 mm to (225.0, 2.58)
- moved C205 243.1 mm to (220.3, 5.53)
- moved R208 243.0 mm to (220.7, 44.3), turned to 180 degrees
- moved R203 225.1 mm to (207.8, 46.0), turned to 180 degrees
- moved R202 221.9 mm to (207.8, 43.9), turned to 180 degrees
- moved R204 217.9 mm to (195.3, 43.1)
- moved R201 217.1 mm to (207.8, 41.9), turned to 180 degrees
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Routing:
- net /USB/USB_5V: track 1.96 -> 96.0 mm, vias 0 -> 1
- net Net-(C1006-Pad1): track 0.00 -> 91.2 mm
- net +5V: track 188.5 -> 278.1 mm, vias 0 -> 2
- net Net-(C1007-Pad1): track 0.00 -> 84.2 mm
- net Net-(U1002-Pad3): track 0.00 -> 80.6 mm, vias 0 -> 2
- net /USB/USBD+: track 0.00 -> 73.4 mm
- net /USB/USBD-: track 0.00 -> 73.4 mm
- net Net-(R1003-Pad2): track 0.00 -> 68.9 mm, vias 0 -> 2
- net Net-(R1007-Pad2): track 0.00 -> 54.8 mm, vias 0 -> 2
- net /USB/USBD1+: track 0.00 -> 39.6 mm
- net /USB/USBD1-: track 0.00 -> 38.8 mm
- net /USB/USB_3V3: track 2.33 -> 37.5 mm, vias 0 -> 1
- net /USB/USBD2-: track 0.00 -> 34.6 mm
- net /USB/USBD2+: track 0.00 -> 34.3 mm
- net Net-(R1006-Pad2): track 0.00 -> 25.5 mm, vias 0 -> 2
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Other:
- net class USB: clearance 0.2 -> 0.1016; trace_width 0.45 -> 0.175006
- board text added: "Slot 0"
- board text added: "Slot 2"
- board text added: "Slot 3"

Commit message: Wired up UART and expansion slots.
Parts:
- moved R1110 305.6 mm to (182.1, 4.34)
- moved R1108 305.6 mm to (179.1, 1.11)
- moved C804 261.2 mm to (159.2, 67.5)
- moved C802 255.3 mm to (159.2, 63.7), turned to 270 degrees
- moved C801 251.7 mm to (159.2, 59.7), turned to 90 degrees
- moved C803 251.6 mm to (162.4, 56.2), turned to 180 degrees
- moved C805 238.0 mm to (171.3, 59.0), turned to 90 degrees
- moved U801 237.0 mm to (165.5, 62.7), turned to 0 degrees
- moved TP102 211.0 mm to (191.8, 162.6)
- moved TP101 210.1 mm to (191.8, 167.6)
- moved TP104 210.0 mm to (186.7, 162.6)
- moved TP103 209.1 mm to (186.7, 167.6)
- moved TP105 206.4 mm to (181.6, 162.6)
- moved BT1201 94.7 mm to (247.8, 190.1)
- moved J701 70.8 mm to (160.8, 182.2)
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Routing:
- net +5V: track 278.1 -> 716.5 mm, vias 2 -> 9
- net /~CS0: track 0.00 -> 356.5 mm, vias 0 -> 1
- net /~IRQ0: track 0.00 -> 353.0 mm, vias 0 -> 1
- net /~CS1: track 0.00 -> 327.9 mm, vias 0 -> 1
- net /~IRQ1: track 0.00 -> 325.6 mm, vias 0 -> 1
- net /~IRQ2: track 0.00 -> 282.7 mm
- net /~CS2: track 0.00 -> 278.2 mm
- net /I2C_SCL: track 64.3 -> 337.1 mm, vias 0 -> 2
- net /I2C_SDA: track 64.0 -> 332.6 mm, vias 0 -> 2
- net /~CS3: track 0.00 -> 259.5 mm
- net /~IRQ3: track 0.00 -> 259.4 mm
- net /~RESET: track 63.7 -> 248.8 mm, vias 0 -> 2
- net /~IRQ7: track 0.00 -> 184.4 mm, vias 0 -> 2
- net /SPI_CLK: track 63.7 -> 215.1 mm, vias 0 -> 1
- net /SPI_COPI: track 63.7 -> 214.9 mm, vias 0 -> 1
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